File: docs/schematics/nostos/nostos-wiring.kicad_sch (KiCad schematic)
At the start: 18 parts, among them SW1 BTN1 SPEED UP, SW2 BTN2 SPEED DOWN, SW3 BTN3 STOP REQUEST, SW4 BTN4 LOCAL / MSG_NONE, U1 NUCLEO-F411RE, U2 ESP32-S3 BLE MESH BRIDGE, U3 VS1003B AUDIO DECODER, U4 MPU6050 (RIDER TAIL, ON), U5 DHT11 (RIDER MID, ON)

Commit message: refactor: simplify NOSTOS firmware protocol
Parts:
- U4: value MPU6050 (RIDER TAIL, ON) -> MPU6050 (RIDER NODE 3, ON)
- U5: value DHT11 (RIDER MID, ON) -> DHT11 (RIDER NODE 2, ON)
Other:
- note added: "Rider Node 1: Base configuration (SSD1306 + VS1003B)"
- note added: "Rider Node 2: Base + DHT11 (ON)"
- note added: "Rider Node 3: Base + MPU6050 (ON)"
- note removed: "Rider Head: Base configuration (SSD1306 + VS1003B)"
- note removed: "Rider Mid: Base + DHT11 (ON)"
- note removed: "Rider Tail: Base + MPU6050 (ON)"
Changed lines of the file:
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@@
 		(comment 2 "STM32 NUCLEO-F411RE / 3.3V logic / Common GND")
 		(comment 3 "Documentation schematic - verify breakout module power ratings")
-		(comment 4 "Rider Head=Base, Mid=Base+DHT11, Tail=Base+MPU6050")
+		(comment 4 "Node 1=Base, Node 2=Base+DHT11, Node 3=Base+MPU6050")
 	)
 	(text "VS1003B supply is breakout-dependent. Confirm its VIN rating; all signal levels remain 3.3V."
@@
 		)
 	)
-	(text "Rider Mid: Base + DHT11 (ON)"
+	(text "Rider Node 2: Base + DHT11 (ON)"
 		(exclude_from_sim no)
 		(at 254 240.03 0)
@@
 		)
 	)
-	(text "Rider Tail: Base + MPU6050 (ON)"
+	(text "Rider Node 3: Base + MPU6050 (ON)"
 		(exclude_from_sim no)
 		(at 254 245.11 0)
@@
 		)
 	)
-	(text "Rider Head: Base configuration (SSD1306 + VS1003B)"
+	(text "Rider Node 1: Base configuration (SSD1306 + VS1003B)"
 		(exclude_from_sim no)
 		(at 254 234.95 0)
@@
 			)
 		)
-		(property "Value" "MPU6050 (RIDER TAIL, ON)"
+		(property "Value" "MPU6050 (RIDER NODE 3, ON)"
 			(at 63.5 184.15 0)
 			(show_name no)
@@
 			)
 		)
-		(property "Value" "DHT11 (RIDER MID, ON)"
+		(property "Value" "DHT11 (RIDER NODE 2, ON)"
 			(at 132.08 186.69 0)
 			(show_name no)
